File: matrix.kicad_sch (KiCad schematic)
At the start: 0 parts

Commit message: Created matrix.
Parts:
- added D1, D10, D11, D12, D13, D14, D15, D16, D17, D18, D19, D2, D20, D3, D4, D5, D6, D7, D8, D9: SOD-123, Diodes_SMD:D_SOD-123, symbol Device:D_Small
- added MX1, MX10, MX11, MX12, MX13, MX14, MX15, MX16, MX17, MX18, MX19, MX2, MX20, MX21, MX22, MX23, MX3, MX4, MX5, MX6, MX7, MX8, MX9: MX-NoLED, symbol MX_Alps_Hybrid:MX-NoLED
Connections:
- new net: D10.1 (K), D11.1 (K), D12.1 (K), D9.1 (K)
- new net: D10.2 (A), MX18.2 (ROW)
- new net: D5.1 (K), D6.1 (K), D7.1 (K), D8.1 (K)
- new net: D5.2 (A), MX13.2 (ROW)
- new net: D11.2 (A), MX19.2 (ROW)
- new net: D18.2 (A), MX2.2 (ROW)
- new net: D12.2 (A), MX20.2 (ROW), MX23.2 (ROW)
- new net: D16.2 (A), MX8.2 (ROW)
- new net: D1.1 (K), D2.1 (K), D3.1 (K), D4.1 (K)
- new net: D3.2 (A), MX10.2 (ROW)
- new net: D13.1 (K), D14.1 (K), D15.1 (K), D16.1 (K)
- new net: D15.2 (A), MX7.2 (ROW)
- new net: D19.2 (A), MX3.2 (ROW)
- new net: D7.2 (A), MX15.2 (ROW)
- new net: D17.2 (A), MX1.2 (ROW)
- new net: D9.2 (A), MX17.2 (ROW), MX21.2 (ROW)
- new net: D20.2 (A), MX4.2 (ROW)
- new net: D2.2 (A), MX11.2 (ROW)
- new net: D8.2 (A), MX16.2 (ROW)
- new net: D14.2 (A), MX6.2 (ROW)
- new net: D1.2 (A), MX12.2 (ROW), MX22.2 (ROW)
- new net: D6.2 (A), MX14.2 (ROW)
- new net: D17.1 (K), D18.1 (K), D19.1 (K), D20.1 (K)
- new net: D4.2 (A), MX9.2 (ROW)
- new net: D13.2 (A), MX5.2 (ROW)
- new net COL0: MX1.1 (COL), MX13.1 (COL), MX17.1 (COL), MX21.1 (COL), MX5.1 (COL), MX9.1 (COL)
- new net COL1: MX10.1 (COL), MX14.1 (COL), MX18.1 (COL), MX2.1 (COL), MX6.1 (COL)
- new net COL2: MX11.1 (COL), MX15.1 (COL), MX19.1 (COL), MX3.1 (COL), MX7.1 (COL)
- new net COL3: MX12.1 (COL), MX16.1 (COL), MX20.1 (COL), MX22.1 (COL), MX23.1 (COL), MX4.1 (COL), MX8.1 (COL)
