File: rgb.kicad_sch (KiCad schematic)
At the start: 0 parts

Commit message: creating led matrix.
Parts:
- added D21, D22, D23, D24, D25, D26, D27, D28: SK6805, LED_SMD:LED_SK6805_PLCC4_2.4x2.7mm_P1.3mm, symbol LED:SK6805
Connections:
- new net: D21.3 (DIN), D22.1 (DOUT)
- new net: D22.3 (DIN), D23.1 (DOUT)
- new net: D24.3 (DIN), D25.1 (DOUT)
- new net: D25.3 (DIN), D26.1 (DOUT)
- new net: D23.3 (DIN), D24.1 (DOUT)
- new net: D27.3 (DIN), D28.1 (DOUT)
- new net: D26.3 (DIN), D27.1 (DOUT)
